File: _autosave-AWG.kicad_pcb (KiCad board)
At the start: 2 copper layers, 73 parts, among them J1001 Conn_01x03, J1002 Conn_01x05, J1003 Conn_01x06, J1004 Conn_01x06, J2 Conn afficheur, J5 SMA, J6 SMA, Q1001 NTE2633, Q1002 NTE2634, U1001 L7812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

Commit message: 3D shapes added
Parts:
- added U1: Pico, Pi_Pico:RPi_Pico_SMD_TH, F.Cu at (186.1, 96.0)
- U1002, U1004: footprint Package_TO_SOT_SMD:TO-263-2 -> Package_TO_SOT_SMD:TO-252-2
