File: AWG.sch (KiCad schematic (older format))
At the start: 92 parts, among them J1001 Conn_01x03, J1002 Conn_01x05, J1003 Conn_01x06, J1004 Conn_01x06, J1005 Conn_01x01, J1006 Conn_01x01, J1007 Conn_01x01, J1008 Conn_01x01, J1009 Conn_01x01, J1010 Conn_01x01, J1011 Conn_01x01, J1012 Conn_01x01, J1013 Conn_01x05, J2 Conn afficheur, J5 SMA, J6 SMA, J7 BNC, Q1001 NTE2633, Q1002 NTE2634, SW1 Reset, SW2 Encodeur sur façade, SW3 Next, SW4 Previous, SW5 AC/DC, SW6 50R/Low Z, U1 Pico, U1001 L7812, U1002 L7912, U1003 L7805, U1004 L7905, U3 AD8055ARZ

Commit message: minor cosmetic details.Bypass cap changed
Parts:
- C6: footprint Capacitor_THT:C_Radial_D10.0mm_H16.0mm_P5.00mm -> Capacitor_SMD:C_1812_4532Metric_Pad1.57x3.40mm_HandSolder
Changed lines of the file:
@@
 F 0 "C6" V 5821 4450 50  0000 C CNN
 F 1 "1mF" V 5912 4450 50  0000 C CNN
-F 2 "Capacitor_THT:C_Radial_D10.0mm_H16.0mm_P5.00mm" H 6050 4450 50  0001 C CNN
+F 2 "Capacitor_SMD:C_1812_4532Metric_Pad1.57x3.40mm_HandSolder" H 6050 4450 50  0001 C CNN
 F 3 "~" H 6050 4450 50  0001 C CNN
 	1    6050 4450
